Commit message: Updated location of link 1

File: fanuc_r2000ic_support/urdf/r2000ic_165f_macro.xacro (robot description, xacro)
@@ -111,5 +111,5 @@
     <!-- joints: main serial chain -->
     <joint name="${prefix}joint_1" type="revolute">
-      <origin xyz="0 0 0.670" rpy="0 0 0"/>
+      <origin xyz="0 0 0" rpy="0 0 0"/>
       <parent link="${prefix}base_link"/>
       <child link="${prefix}link_1"/>
@@ -118,5 +118,5 @@
     </joint>
     <joint name="${prefix}joint_2" type="revolute">
-      <origin xyz="0.312 0 0" rpy="0 0 0"/>
+      <origin xyz="0.312 0 0.670" rpy="0 0 0"/>
       <parent link="${prefix}link_1"/>
       <child link="${prefix}link_2"/>
