Commit message: Renamed from r2000ic16f to r2000ic_165f

File: fanuc_r2000ic_support/urdf/r2000ic_165f.xacro (robot description, xacro)
@@ -1,5 +1,5 @@
 <?xml version="1.0" ?>
-<robot name="fanuc_r2000ic165f" xmlns:xacro="http://wiki.ros.org/xacro">
+<robot name="fanuc_r2000ic_165f" xmlns:xacro="http://wiki.ros.org/xacro">
   <xacro:include filename="$(find fanuc_r2000ic_support)/urdf/r2000ic_165f_macro.xacro"/>
-  <xacro:fanuc_r2000ic165f prefix=""/>
+  <xacro:fanuc_r2000ic_165f prefix=""/>
 </robot>

File: fanuc_r2000ic_support/urdf/r2000ic_165f_macro.xacro (robot description, xacro)
@@ -2,5 +2,5 @@
 <robot xmlns:xacro="http://wiki.ros.org/xacro">
   <xacro:include filename="$(find fanuc_resources)/urdf/common_materials.xacro"/>
-  <xacro:macro name="fanuc_r2000ic165f" params="prefix">
+  <xacro:macro name="fanuc_r2000ic_165f" params="prefix">
     <!-- links: main serial chain -->
     <link name="${prefix}base_link">
@@ -8,5 +8,5 @@
         <origin xyz="0 0 0" rpy="0 0 0"/>
         <geometry>
-          <mesh filename="package://fanuc_r2000ic_support/meshes/r2000ic165f/visual/base_link.stl"/>
+          <mesh filename="package://fanuc_r2000ic_support/meshes/r2000ic_165f/visual/base_link.stl"/>
         </geometry>
         <xacro:material_fanuc_gray40 />
@@ -15,5 +15,5 @@
         <origin xyz="0 0 0" rpy="0 0 0"/>
         <geometry>
-          <mesh filename="package://fanuc_r2000ic_support/meshes/r2000ic165f/collision/base_link.stl"/>
+          <mesh filename="package://fanuc_r2000ic_support/meshes/r2000ic_165f/collision/base_link.stl"/>
         </geometry>
       </collision>
@@ -23,5 +23,5 @@
         <origin xyz="0 0 0" rpy="0 0 0"/>
         <geometry>
-          <mesh filename="package://fanuc_r2000ic_support/meshes/r2000ic165f/visual/link_1.stl"/>
+          <mesh filename="package://fanuc_r2000ic_support/meshes/r2000ic_165f/visual/link_1.stl"/>
         </geometry>
         <xacro:material_fanuc_yellow />
@@ -30,5 +30,5 @@
         <origin xyz="0 0 0" rpy="0 0 0"/>
         <geometry>
-          <mesh filename="package://fanuc_r2000ic_support/meshes/r2000ic165f/collision/link_1.stl"/>
+          <mesh filename="package://fanuc_r2000ic_support/meshes/r2000ic_165f/collision/link_1.stl"/>
         </geometry>
       </collision>
@@ -38,5 +38,5 @@
         <origin xyz="0 0 0" rpy="0 0 0"/>
         <geometry>
-          <mesh filename="package://fanuc_r2000ic_support/meshes/r2000ic165f/visual/link_2.stl"/>
+          <mesh filename="package://fanuc_r2000ic_support/meshes/r2000ic_165f/visual/link_2.stl"/>
         </geometry>
         <xacro:material_fanuc_yellow />
@@ -45,5 +45,5 @@
         <origin xyz="0 0 0" rpy="0 0 0"/>
         <geometry>
-          <mesh filename="package://fanuc_r2000ic_support/meshes/r2000ic165f/collision/link_2.stl"/>
+          <mesh filename="package://fanuc_r2000ic_support/meshes/r2000ic_165f/collision/link_2.stl"/>
         </geometry>
       </collision>
@@ -53,5 +53,5 @@
         <origin xyz="0 0 0" rpy="0 0 0"/>
         <geometry>
-          <mesh filename="package://fanuc_r2000ic_support/meshes/r2000ic165f/visual/link_3.stl"/>
+          <mesh filename="package://fanuc_r2000ic_support/meshes/r2000ic_165f/visual/link_3.stl"/>
         </geometry>
         <xacro:material_fanuc_yellow />
@@ -60,5 +60,5 @@
         <origin xyz="0 0 0" rpy="0 0 0"/>
         <geometry>
-          <mesh filename="package://fanuc_r2000ic_support/meshes/r2000ic165f/collision/link_3.stl"/>
+          <mesh filename="package://fanuc_r2000ic_support/meshes/r2000ic_165f/collision/link_3.stl"/>
         </geometry>
       </collision>
@@ -68,5 +68,5 @@
         <origin xyz="0 0 0" rpy="0 0 0"/>
         <geometry>
-          <mesh filename="package://fanuc_r2000ic_support/meshes/r2000ic165f/visual/link_4.stl"/>
+          <mesh filename="package://fanuc_r2000ic_support/meshes/r2000ic_165f/visual/link_4.stl"/>
         </geometry>
         <xacro:material_fanuc_yellow />
@@ -75,5 +75,5 @@
         <origin xyz="0 0 0" rpy="0 0 0"/>
         <geometry>
-          <mesh filename="package://fanuc_r2000ic_support/meshes/r2000ic165f/collision/link_4.stl"/>
+          <mesh filename="package://fanuc_r2000ic_support/meshes/r2000ic_165f/collision/link_4.stl"/>
         </geometry>
       </collision>
@@ -83,5 +83,5 @@
         <origin xyz="0 0 0" rpy="0 0 0"/>
         <geometry>
-          <mesh filename="package://fanuc_r2000ic_support/meshes/r2000ic165f/visual/link_5.stl"/>
+          <mesh filename="package://fanuc_r2000ic_support/meshes/r2000ic_165f/visual/link_5.stl"/>
         </geometry>
         <xacro:material_fanuc_yellow />
@@ -90,5 +90,5 @@
         <origin xyz="0 0 0" rpy="0 0 0"/>
         <geometry>
-          <mesh filename="package://fanuc_r2000ic_support/meshes/r2000ic165f/collision/link_5.stl"/>
+          <mesh filename="package://fanuc_r2000ic_support/meshes/r2000ic_165f/collision/link_5.stl"/>
         </geometry>
       </collision>
@@ -98,5 +98,5 @@
         <origin xyz="0 0 0" rpy="0 0 0"/>
         <geometry>
-          <mesh filename="package://fanuc_r2000ic_support/meshes/r2000ic165f/visual/link_6.stl"/>
+          <mesh filename="package://fanuc_r2000ic_support/meshes/r2000ic_165f/visual/link_6.stl"/>
         </geometry>
         <xacro:material_fanuc_black />
@@ -105,5 +105,5 @@
         <origin xyz="0 0 0" rpy="0 0 0"/>
         <geometry>
-          <mesh filename="package://fanuc_r2000ic_support/meshes/r2000ic165f/collision/link_6.stl"/>
+          <mesh filename="package://fanuc_r2000ic_support/meshes/r2000ic_165f/collision/link_6.stl"/>
         </geometry>
       </collision>
